File: board/E155 Breadboard Adapter/MicroPs Cobbler.kicad_sch (KiCad schematic)
At the start: 3 parts, among them J1 Conn_01x20, J2 40-pin Ribbon Cable Connector, J3 Conn_01x20

Commit message: Board updates for FA24
Removed specific text on the board which references a year and changed it to a version number. Also updated the libraries and KiCad files to resolve design check issues.
Other:
- title: E155 FA23 Breadboard Adapter -> E155 Breadboard Adapter
Changed lines of the file:
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@@
   (paper "A4")
   (title_block
-    (title "E155 FA23 Breadboard Adapter")
+    (title "E155 Breadboard Adapter")
     (rev "v4")
     (company "Harvey Mudd College")
@@
     (pin "9")
     (instances
-      (project "MicroPs Cobbler v3"
+      (project "MicroPs Cobbler"
         (path "/55992e35-fe7b-468a-9b7a-1e4dc931b904"
           (reference "J3") (unit 1)
@@
     (pin "9")
     (instances
-      (project "MicroPs Cobbler v3"
+      (project "MicroPs Cobbler"
         (path "/55992e35-fe7b-468a-9b7a-1e4dc931b904"
           (reference "J1") (unit 1)
@@
     (pin "9")
     (instances
-      (project "MicroPs Cobbler v3"
+      (project "MicroPs Cobbler"
         (path "/55992e35-fe7b-468a-9b7a-1e4dc931b904"
           (reference "J2") (unit 1)
